Commit message: build commit

File: motoman_resources/urdf/common_materials.xacro (robot description, xacro)
@@ -1,26 +1,24 @@
 <?xml version="1.0" ?>
 <robot xmlns:xacro="http://ros.org/wiki/xacro">
+  <!-- Include the color definitions -->
   <xacro:include filename="$(find motoman_resources)/urdf/common_colors.xacro"/>
-  <xacro:macro name="material_yaskawa_blue">
-    <material name="">
-      <color rgba="${color_yaskawa_blue}"/>
-    </material>
-  </xacro:macro>
-  <xacro:macro name="material_yaskawa_white">
-    <material name="">
-      <color rgba="${color_yaskawa_white}"/>
-    </material>
-  </xacro:macro>
-  <!-- not an official colour, but used in some old xacro:macros -->
-  <xacro:macro name="material_yaskawa_yellow">
-    <material name="">
-      <color rgba="${color_yaskawa_yellow}"/>
-    </material>
-  </xacro:macro>
-  <!-- not an official colour, but used in some old xacro:macros -->
-  <xacro:macro name="material_yaskawa_silver">
-    <material name="">
-      <color rgba="${color_yaskawa_silver}"/>
-    </material>
+  <!-- Include the material definitions -->
+  <xacro:include filename="$(find motoman_resources)/urdf/common_materials.xacro"/>
+  <!-- Include the Motoman GP7 XACRO -->
+  <xacro:include filename="$(find motoman_gp7_description)/urdf/motoman_gp7.xacro"/>
+  <!-- Include the Kiwi Cell XACRO -->
+  <xacro:include filename="$(find kiwi_cell_description)/urdf/kiwi_cell.xacro"/>
+  <!-- Define the combined robot -->
+  <xacro:macro name="combined_robot" params="prefix">
+    <!-- Motoman GP7 robot -->
+    <xacro:motoman_gp7 prefix="${prefix}"/>
+    <!-- Kiwi Cell robot -->
+    <xacro:kiwi_cell prefix="${prefix}"/>
+    <!-- Example: Adding a transform between the two robot parts -->
+    <joint name="${prefix}motoman_kiwi_transform" type="fixed">
+      <origin xyz="1.0 0 0" rpy="0 0 0"/>
+      <parent link="${prefix}link_6_t"/>
+      <child link="${prefix}base_link"/>
+    </joint>
   </xacro:macro>
 </robot>
